File: Templates/STM32_NUCELO_Shield_2_Layer/template.kicad_sch (KiCad schematic)
At the start: 0 parts

Commit message: schematic update - added title
Other:
- note added: "TITLE"
Changed lines of the file:
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@@
 	(paper "A4")
 	(title_block
-		(date "2025-12-26")
+		(date "2025-12-27")
 		(rev "${REVISION}")
 		(company "Author:")
 	)
+	(text "TITLE"
+		(exclude_from_sim no)
+		(at 12.7 24.13 0)
+		(effects
+			(font
+				(size 12 12)
+				(thickness 4.8)
+				(bold yes)
+			)
+			(justify left)
+		)
+	)
 	(sheet_instances
